Commit message: ros2: widen canonical G1 Gazebo world for V2.1

File: ros2_ws/src/dynnav_nav2_benchmark/worlds/g1_parallel_corridor.sdf.xacro (robot description, xacro)
@@ -17,10 +17,4 @@
       <diffuse>0.8 0.8 0.8 1</diffuse>
       <specular>0.8 0.8 0.8 1</specular>
-      <attenuation>
-        <range>1000</range>
-        <constant>0.9</constant>
-        <linear>0.01</linear>
-        <quadratic>0.001</quadratic>
-      </attenuation>
       <direction>-0.5 0.1 -0.9</direction>
     </light>
@@ -38,15 +32,15 @@
     </model>
     <model name="boundary_left">
-      <static>1</static><pose>0.075 2.5 0.5 0 0 0</pose>
+      <static>1</static><pose>0.075 3.2 0.5 0 0 0</pose>
       <link name="link">
-        <collision name="collision"><geometry><box><size>0.15 5.0 1.0</size></box></geometry></collision>
-        <visual name="visual"><geometry><box><size>0.15 5.0 1.0</size></box></geometry></visual>
+        <collision name="collision"><geometry><box><size>0.15 6.4 1.0</size></box></geometry></collision>
+        <visual name="visual"><geometry><box><size>0.15 6.4 1.0</size></box></geometry></visual>
       </link>
     </model>
     <model name="boundary_right">
-      <static>1</static><pose>6.925 2.5 0.5 0 0 0</pose>
+      <static>1</static><pose>6.925 3.2 0.5 0 0 0</pose>
       <link name="link">
-        <collision name="collision"><geometry><box><size>0.15 5.0 1.0</size></box></geometry></collision>
-        <visual name="visual"><geometry><box><size>0.15 5.0 1.0</size></box></geometry></visual>
+        <collision name="collision"><geometry><box><size>0.15 6.4 1.0</size></box></geometry></collision>
+        <visual name="visual"><geometry><box><size>0.15 6.4 1.0</size></box></geometry></visual>
       </link>
     </model>
@@ -59,5 +53,5 @@
     </model>
     <model name="boundary_top">
-      <static>1</static><pose>3.5 4.925 0.5 0 0 0</pose>
+      <static>1</static><pose>3.5 6.325 0.5 0 0 0</pose>
       <link name="link">
         <collision name="collision"><geometry><box><size>7.0 0.15 1.0</size></box></geometry></collision>
@@ -66,9 +60,9 @@
     </model>
     <model name="central_island">
-      <static>1</static><pose>3.5 2.5 0.5 0 0 0</pose>
+      <static>1</static><pose>3.5 3.2 0.5 0 0 0</pose>
       <link name="link">
-        <collision name="collision"><geometry><box><size>4.0 1.6 1.0</size></box></geometry></collision>
+        <collision name="collision"><geometry><box><size>4.0 2.0 1.0</size></box></geometry></collision>
         <visual name="visual">
-          <geometry><box><size>4.0 1.6 1.0</size></box></geometry>
+          <geometry><box><size>4.0 2.0 1.0</size></box></geometry>
           <material><ambient>0.35 0.35 0.35 1</ambient><diffuse>0.35 0.35 0.35 1</diffuse></material>
         </visual>
